Commit message: updated urdf files

File: urdf/innok_heros_3w.xacro (robot description, xacro)
@@ -10,5 +10,5 @@
 THIS SOFTWARE IS PROVIDED BY THE COPYRIGHT HOLDERS AND CONTRIBUTORS "AS IS" AND ANY EXPRESS OR IMPLIED WARRANTIES, INCLUDING, BUT NOT LIMITED TO, THE IMPLIED WARRANTIES OF MERCHANTABILITY AND FITNESS FOR A PARTICULAR PURPOSE ARE DISCLAIMED. IN NO EVENT SHALL THE COPYRIGHT HOLDER OR CONTRIBUTORS BE LIABLE FOR ANY DIRECT, INDIRECT, INCIDENTAL, SPECIAL, EXEMPLARY, OR CONSEQUENTIAL DAMAGES (INCLUDING, BUT NOT LIMITED TO, PROCUREMENT OF SUBSTITUTE GOODS OR SERVICES; LOSS OF USE, DATA, OR PROFITS; OR BUSINESS INTERRUPTION) HOWEVER CAUSED AND ON ANY THEORY OF LIABILITY, WHETHER IN CONTRACT, STRICT LIABILITY, OR TORT (INCLUDING NEGLIGENCE OR OTHERWISE) ARISING IN ANY WAY OUT OF THE USE OF THIS SOFTWARE, EVEN IF ADVISED OF THE POSSIBILITY OF SUCH DAMAGE.
 -->
-<robot name="innok_heros_3" xmlns:xacro="http://ros.org/wiki/xacro">
+<robot name="innok_heros_3" xmlns:xacro="http://www.ros.org/wiki/xacro">
   <xacro:property name="PI" value="3.1415926535897931"/>
   <xacro:property name="wheel_radius" value="0.160" />
@@ -23,14 +23,15 @@
   <xacro:include filename="$(find innok_heros_description)/urdf/modules/heros_battery.xacro" />
   <xacro:include filename="$(find innok_heros_description)/urdf/modules/heros_mounting_plate.xacro" />
+  <xacro:include filename="$(find innok_heros_description)/urdf/modules/heros_pan.xacro" />
   <xacro:include filename="$(find innok_heros_description)/urdf/ROS/heros_joint_pub.xacro" />
   <xacro:include filename="$(find innok_heros_description)/urdf/ROS/heros_diff_drive.xacro" />
   <!-- heros modules-->
-  <heros_base_link   							/>
-  <heros_drive   	  front_rear='rear'     dx='0.018' flip_z='1'/>
-  <heros_caster  	 	         	dx='0.637'		/>
-  <heros_battery 	  name='battery_box'    dx='0.336'		/>
-  <heros_mounting_plate   wheels='3'		dx='-0.02'		/>
+  <xacro:heros_base_link/>
+  <xacro:heros_drive front_rear='rear' dx='0.018' flip_z='1'/>
+  <xacro:heros_caster dx='0.637'/>
+  <xacro:heros_battery name='battery_box' dx='0.336'/>
+  <xacro:heros_mounting_plate wheels='3' dx='-0.02'/>
   <!-- heros ROS plugins-->
-  <heros_joint_pub joints='joint_base_wheel_rear_left, joint_base_wheel_rear_right, caster_bot_joint, caster_wheel_joint'					/>
-  <heros_diff_drive 							/>
+  <xacro:heros_joint_pub joints='joint_base_wheel_rear_left, joint_base_wheel_rear_right, caster_bot_joint, caster_wheel_joint'					/>
+  <xacro:heros_diff_drive 							/>
 </robot>

File: urdf/innok_heros_3wtractor.xacro (robot description, xacro)
@@ -10,5 +10,5 @@
 THIS SOFTWARE IS PROVIDED BY THE COPYRIGHT HOLDERS AND CONTRIBUTORS "AS IS" AND ANY EXPRESS OR IMPLIED WARRANTIES, INCLUDING, BUT NOT LIMITED TO, THE IMPLIED WARRANTIES OF MERCHANTABILITY AND FITNESS FOR A PARTICULAR PURPOSE ARE DISCLAIMED. IN NO EVENT SHALL THE COPYRIGHT HOLDER OR CONTRIBUTORS BE LIABLE FOR ANY DIRECT, INDIRECT, INCIDENTAL, SPECIAL, EXEMPLARY, OR CONSEQUENTIAL DAMAGES (INCLUDING, BUT NOT LIMITED TO, PROCUREMENT OF SUBSTITUTE GOODS OR SERVICES; LOSS OF USE, DATA, OR PROFITS; OR BUSINESS INTERRUPTION) HOWEVER CAUSED AND ON ANY THEORY OF LIABILITY, WHETHER IN CONTRACT, STRICT LIABILITY, OR TORT (INCLUDING NEGLIGENCE OR OTHERWISE) ARISING IN ANY WAY OUT OF THE USE OF THIS SOFTWARE, EVEN IF ADVISED OF THE POSSIBILITY OF SUCH DAMAGE.
 -->
-<robot name="innok_heros_3w" xmlns:xacro="http://ros.org/wiki/xacro">
+<robot name="innok_heros_3wtractor" xmlns:xacro="http://www.ros.org/wiki/xacro">
   <xacro:property name="PI" value="3.1415926535897931"/>
   <xacro:property name="wheel_radius" value="0.200" />

File: urdf/innok_heros_4w.xacro (robot description, xacro)
@@ -10,9 +10,11 @@
 THIS SOFTWARE IS PROVIDED BY THE COPYRIGHT HOLDERS AND CONTRIBUTORS "AS IS" AND ANY EXPRESS OR IMPLIED WARRANTIES, INCLUDING, BUT NOT LIMITED TO, THE IMPLIED WARRANTIES OF MERCHANTABILITY AND FITNESS FOR A PARTICULAR PURPOSE ARE DISCLAIMED. IN NO EVENT SHALL THE COPYRIGHT HOLDER OR CONTRIBUTORS BE LIABLE FOR ANY DIRECT, INDIRECT, INCIDENTAL, SPECIAL, EXEMPLARY, OR CONSEQUENTIAL DAMAGES (INCLUDING, BUT NOT LIMITED TO, PROCUREMENT OF SUBSTITUTE GOODS OR SERVICES; LOSS OF USE, DATA, OR PROFITS; OR BUSINESS INTERRUPTION) HOWEVER CAUSED AND ON ANY THEORY OF LIABILITY, WHETHER IN CONTRACT, STRICT LIABILITY, OR TORT (INCLUDING NEGLIGENCE OR OTHERWISE) ARISING IN ANY WAY OUT OF THE USE OF THIS SOFTWARE, EVEN IF ADVISED OF THE POSSIBILITY OF SUCH DAMAGE.
 -->
-<robot name="innok_heros_4w" xmlns:xacro="http://ros.org/wiki/xacro">
+<robot name="innok_heros_4w" xmlns:xacro="http://www.ros.org/wiki/xacro">
   <xacro:property name="PI" value="3.1415926535897931"/>
   <xacro:property name="wheel_radius" value="0.160" />
   <xacro:property name="wheel_width"  value="0.160" />
   <xacro:property name="wheel_mass"   value="5.4" />
+  <xacro:property name="wheel_seperation" value="0.580" />
+  <xacro:property name="camera_link"   value="0.05" />
   <xacro:include filename="$(find innok_heros_description)/urdf/modules/heros_base_link.xacro"/>
   <xacro:include filename="$(find innok_heros_description)/urdf/modules/heros_wheel.xacro"/>

File: urdf/innok_heros_4wtractor.xacro (robot description, xacro)
@@ -10,5 +10,5 @@
 THIS SOFTWARE IS PROVIDED BY THE COPYRIGHT HOLDERS AND CONTRIBUTORS "AS IS" AND ANY EXPRESS OR IMPLIED WARRANTIES, INCLUDING, BUT NOT LIMITED TO, THE IMPLIED WARRANTIES OF MERCHANTABILITY AND FITNESS FOR A PARTICULAR PURPOSE ARE DISCLAIMED. IN NO EVENT SHALL THE COPYRIGHT HOLDER OR CONTRIBUTORS BE LIABLE FOR ANY DIRECT, INDIRECT, INCIDENTAL, SPECIAL, EXEMPLARY, OR CONSEQUENTIAL DAMAGES (INCLUDING, BUT NOT LIMITED TO, PROCUREMENT OF SUBSTITUTE GOODS OR SERVICES; LOSS OF USE, DATA, OR PROFITS; OR BUSINESS INTERRUPTION) HOWEVER CAUSED AND ON ANY THEORY OF LIABILITY, WHETHER IN CONTRACT, STRICT LIABILITY, OR TORT (INCLUDING NEGLIGENCE OR OTHERWISE) ARISING IN ANY WAY OUT OF THE USE OF THIS SOFTWARE, EVEN IF ADVISED OF THE POSSIBILITY OF SUCH DAMAGE.
 -->
-<robot name="innok_heros_4w" xmlns:xacro="http://ros.org/wiki/xacro">
+<robot name="innok_heros_4wtractor" xmlns:xacro="http://www.ros.org/wiki/xacro">
   <xacro:property name="PI" value="3.1415926535897931"/>
   <xacro:property name="wheel_radius" value="0.200" />

File: urdf/modules/heros_drive.xacro (robot description, xacro)
@@ -12,11 +12,22 @@
 -->
 <robot xmlns:xacro="http://ros.org/wiki/xacro" name="heros_drive">
-<xacro:macro name="heros_drive" params="front_rear dx flip_z">
-  <heros_wheel front_rear="${front_rear}" left_right="left"  flip_y="1"  flip_z="${flip_z}"/>
-  <heros_wheel front_rear="${front_rear}" left_right="right" flip_y="-1" flip_z="${flip_z}"/>
+<xacro:macro name="heros_drive" params="front_rear dx flip_z wheel_kind:=0">
+  <xacro:if value="${wheel_kind == 0}">
+    <xacro:heros_wheel front_rear="${front_rear}" left_right="left"  flip_y="1"  flip_z="${flip_z}"/>
+    <xacro:heros_wheel front_rear="${front_rear}" left_right="right" flip_y="-1" flip_z="${flip_z}"/>
+  </xacro:if>
+  <xacro:if value="${wheel_kind == 1}">
+    <xacro:heros_wheel_tractor front_rear="${front_rear}" left_right="left"  flip_y="1"  flip_z="${flip_z}"/>
+    <xacro:heros_wheel_tractor front_rear="${front_rear}" left_right="right" flip_y="-1" flip_z="${flip_z}"/>
+  </xacro:if>
+  <xacro:if value="${wheel_kind == 2}">
+    <xacro:heros_wheel_tractor_large front_rear="${front_rear}" left_right="left"  flip_y="1"  flip_z="${flip_z}"/>
+    <xacro:heros_wheel_tractor_large front_rear="${front_rear}" left_right="right" flip_y="-1" flip_z="${flip_z}"/>
+  </xacro:if>
   <link name="drive_box_${front_rear}">
     <inertial>
       <origin xyz="0.122 -0.0026 -0.136" rpy="0 0 0" />
-       <mass value="10.6" />
+       <!--mass value="10.6" /-->
+       <mass value="0.5" />
       <inertia ixx="0.316" ixy="0" ixz="0" iyy="0.166" iyz="0" izz="0.307" />
     </inertial>

File: urdf/modules/heros_swing_axle.xacro (robot description, xacro)
@@ -33,5 +33,5 @@
   </link>
   <joint name="swing_axle_top_joint" type="fixed">
-    <origin xyz="${dx} -0.22 -0.2" rpy="0 0 ${PI/2}" />
+    <origin xyz="${dx} -0.215 -0.2" rpy="0 0 ${PI/2}" />
     <parent link="beam_link" />
     <child link="swing_axle_top" />

File: urdf/modules/heros_wheel_tractor.xacro (robot description, xacro)
@@ -11,6 +11,6 @@
 THIS SOFTWARE IS PROVIDED BY THE COPYRIGHT HOLDERS AND CONTRIBUTORS "AS IS" AND ANY EXPRESS OR IMPLIED WARRANTIES, INCLUDING, BUT NOT LIMITED TO, THE IMPLIED WARRANTIES OF MERCHANTABILITY AND FITNESS FOR A PARTICULAR PURPOSE ARE DISCLAIMED. IN NO EVENT SHALL THE COPYRIGHT HOLDER OR CONTRIBUTORS BE LIABLE FOR ANY DIRECT, INDIRECT, INCIDENTAL, SPECIAL, EXEMPLARY, OR CONSEQUENTIAL DAMAGES (INCLUDING, BUT NOT LIMITED TO, PROCUREMENT OF SUBSTITUTE GOODS OR SERVICES; LOSS OF USE, DATA, OR PROFITS; OR BUSINESS INTERRUPTION) HOWEVER CAUSED AND ON ANY THEORY OF LIABILITY, WHETHER IN CONTRACT, STRICT LIABILITY, OR TORT (INCLUDING NEGLIGENCE OR OTHERWISE) ARISING IN ANY WAY OUT OF THE USE OF THIS SOFTWARE, EVEN IF ADVISED OF THE POSSIBILITY OF SUCH DAMAGE.
 -->
-<robot xmlns:xacro="http://ros.org/wiki/xacro" name="heros_wheel">
-<xacro:macro name="heros_wheel" params="front_rear left_right flip_y flip_z">
+<robot xmlns:xacro="http://ros.org/wiki/xacro" name="heros_wheel_tractor">
+<xacro:macro name="heros_wheel_tractor" params="front_rear left_right flip_y flip_z">
   <link name="wheel_${front_rear}_${left_right}">
     <collision>

File: urdf/modules/heros_wheel_tractor_large.xacro (robot description, xacro)
@@ -11,6 +11,6 @@
 THIS SOFTWARE IS PROVIDED BY THE COPYRIGHT HOLDERS AND CONTRIBUTORS "AS IS" AND ANY EXPRESS OR IMPLIED WARRANTIES, INCLUDING, BUT NOT LIMITED TO, THE IMPLIED WARRANTIES OF MERCHANTABILITY AND FITNESS FOR A PARTICULAR PURPOSE ARE DISCLAIMED. IN NO EVENT SHALL THE COPYRIGHT HOLDER OR CONTRIBUTORS BE LIABLE FOR ANY DIRECT, INDIRECT, INCIDENTAL, SPECIAL, EXEMPLARY, OR CONSEQUENTIAL DAMAGES (INCLUDING, BUT NOT LIMITED TO, PROCUREMENT OF SUBSTITUTE GOODS OR SERVICES; LOSS OF USE, DATA, OR PROFITS; OR BUSINESS INTERRUPTION) HOWEVER CAUSED AND ON ANY THEORY OF LIABILITY, WHETHER IN CONTRACT, STRICT LIABILITY, OR TORT (INCLUDING NEGLIGENCE OR OTHERWISE) ARISING IN ANY WAY OUT OF THE USE OF THIS SOFTWARE, EVEN IF ADVISED OF THE POSSIBILITY OF SUCH DAMAGE.
 -->
-<robot xmlns:xacro="http://ros.org/wiki/xacro" name="heros_wheel">
-<xacro:macro name="heros_wheel" params="front_rear left_right flip_y flip_z">
+<robot xmlns:xacro="http://ros.org/wiki/xacro" name="heros_wheel_tractor_large">
+<xacro:macro name="heros_wheel_tractor_large" params="front_rear left_right flip_y flip_z">
   <link name="wheel_${front_rear}_${left_right}">
     <collision>
