Commit message: using predefined pi constant

File: urdf/innok_heros.xacro (robot description, xacro)
@@ -3,6 +3,4 @@
   <xacro:arg name="wheel_kind" default="default" /> <!-- default | tractor | tractor_large -->
   <xacro:arg name="front_kind" default="swing_axle" /> <!-- swing_axle | caster | 4wd -->
-  <!-- constants-->
-  <xacro:include filename="$(find innok_heros_description)/urdf/constants.xacro"/>
   <!-- heros base-->
   <xacro:include filename="$(find innok_heros_description)/urdf/innok_heros_universal.xacro"/>

File: urdf/innok_heros_3w.xacro (robot description, xacro)
@@ -11,5 +11,4 @@
 -->
 <robot name="innok_heros_3" xmlns:xacro="http://www.ros.org/wiki/xacro">
-  <xacro:property name="PI" value="3.1415926535897931"/>
   <xacro:property name="wheel_radius" value="0.160" />
   <xacro:property name="wheel_width"  value="0.160" />

File: urdf/innok_heros_3wtractor.xacro (robot description, xacro)
@@ -11,5 +11,4 @@
 -->
 <robot name="innok_heros_3wtractor" xmlns:xacro="http://www.ros.org/wiki/xacro">
-  <xacro:property name="PI" value="3.1415926535897931"/>
   <xacro:property name="wheel_radius" value="0.200" />
   <xacro:property name="wheel_width"  value="0.100" />

File: urdf/innok_heros_4w.xacro (robot description, xacro)
@@ -11,5 +11,4 @@
 -->
 <robot name="innok_heros_4w" xmlns:xacro="http://www.ros.org/wiki/xacro">
-  <xacro:property name="PI" value="3.1415926535897931"/>
   <xacro:property name="wheel_radius" value="0.160" />
   <xacro:property name="wheel_width"  value="0.160" />

File: urdf/innok_heros_4wtractor.xacro (robot description, xacro)
@@ -11,5 +11,4 @@
 -->
 <robot name="innok_heros_4wtractor" xmlns:xacro="http://www.ros.org/wiki/xacro">
-  <xacro:property name="PI" value="3.1415926535897931"/>
   <xacro:property name="wheel_radius" value="0.200" />
   <xacro:property name="wheel_width"  value="0.100" />

File: urdf/innok_heros_universal.xacro (robot description, xacro)
@@ -16,5 +16,4 @@
   </material>
   <!-- Defining xacro properties -->
-  <xacro:property name="PI" value="3.1415926535897931"/>
   <xacro:property name="wheel_seperation" value="0.580" />
   <xacro:property name="camera_link" value="0.05" />

File: urdf/modules/heros_drive.xacro (robot description, xacro)
@@ -39,5 +39,5 @@
   </link>
   <joint name="drive_box_joint_${front_rear}" type="fixed">
-    <origin xyz="${dx} 0 -0.0065" rpy="0 0 ${PI/2 - PI/2*flip_z }" />
+    <origin xyz="${dx} 0 -0.0065" rpy="0 0 ${pi/2 - pi/2*flip_z }" />
     <parent link="beam_link" />
     <child link="drive_box_${front_rear}" />

File: urdf/modules/heros_swing_axle.xacro (robot description, xacro)
@@ -33,5 +33,5 @@
   </link>
   <joint name="swing_axle_top_joint" type="fixed">
-    <origin xyz="${dx} -0.215 -0.2" rpy="0 0 ${PI/2}" />
+    <origin xyz="${dx} -0.215 -0.2" rpy="0 0 ${pi/2}" />
     <parent link="beam_link" />
     <child link="swing_axle_top" />
@@ -179,5 +179,5 @@
   </joint>
   <joint name="caster_left_joint" type="continuous">
-    <origin xyz="-0.215 -0.055 0" rpy="${-PI/2} ${-PI/2} 0" />
+    <origin xyz="-0.215 -0.055 0" rpy="${-pi/2} ${-pi/2} 0" />
     <parent link="swing_axle_bot" />
     <child link="caster_left" />
@@ -185,5 +185,5 @@
   </joint>
   <joint name="caster_right_joint" type="continuous">
-    <origin xyz="0.215 -0.055 0" rpy="${-PI/2} ${-PI/2} 0" />
+    <origin xyz="0.215 -0.055 0" rpy="${-pi/2} ${-pi/2} 0" />
     <parent link="swing_axle_bot" />
     <child link="caster_right" />

File: urdf/modules/heros_wheel.xacro (robot description, xacro)
@@ -15,5 +15,5 @@
   <link name="wheel_${front_rear}_${left_right}">
     <collision>
-      <origin xyz="0 0.115 0" rpy="${-PI/2} 0 0"/>
+      <origin xyz="0 0.115 0" rpy="${-pi/2} 0 0"/>
       <geometry>
         <cylinder radius="${wheel_radius}" length="${wheel_width}" />
@@ -48,5 +48,5 @@
     <parent link="drive_box_${front_rear}"/>
     <child link="wheel_${front_rear}_${left_right}"/>
-    <origin xyz="0.063 ${flip_y*flip_z * 0.162} -0.184" rpy="0 0 ${PI/2 - PI/2*flip_y*flip_z }"/>
+    <origin xyz="0.063 ${flip_y*flip_z * 0.162} -0.184" rpy="0 0 ${pi/2 - pi/2*flip_y*flip_z }"/>
     <axis xyz="0 ${flip_y * 1} 0" />
   </joint>

File: urdf/modules/heros_wheel_tractor.xacro (robot description, xacro)
@@ -15,5 +15,5 @@
   <link name="wheel_${front_rear}_${left_right}">
     <collision>
-      <origin xyz="0 0.115 0" rpy="${-PI/2} 0 0"/>
+      <origin xyz="0 0.115 0" rpy="${-pi/2} 0 0"/>
       <geometry>
         <cylinder radius="${wheel_radius}" length="${wheel_width}" />
@@ -21,5 +21,5 @@
     </collision>
     <visual>
-      <origin xyz="0 0.115 0" rpy="${-PI/2} 0 0"/>
+      <origin xyz="0 0.115 0" rpy="${-pi/2} 0 0"/>
       <geometry>
         <mesh filename="package://innok_heros_description/meshes/wheel_tractor.STL" />
@@ -48,5 +48,5 @@
     <parent link="drive_box_${front_rear}"/>
     <child link="wheel_${front_rear}_${left_right}"/>
-    <origin xyz="0.063 ${flip_y*flip_z * 0.162} -0.184" rpy="0 0 ${PI/2 - PI/2*flip_y*flip_z }"/>
+    <origin xyz="0.063 ${flip_y*flip_z * 0.162} -0.184" rpy="0 0 ${pi/2 - pi/2*flip_y*flip_z }"/>
     <axis xyz="0 ${flip_y * 1} 0" />
   </joint>

File: urdf/modules/heros_wheel_tractor_large.xacro (robot description, xacro)
@@ -15,5 +15,5 @@
   <link name="wheel_${front_rear}_${left_right}">
     <collision>
-      <origin xyz="0 0.115 0" rpy="${-PI/2} 0 0"/>
+      <origin xyz="0 0.115 0" rpy="${-pi/2} 0 0"/>
       <geometry>
         <cylinder radius="${wheel_radius}" length="${wheel_width}" />
@@ -21,5 +21,5 @@
     </collision>
     <visual>
-      <origin xyz="0 0.115 0" rpy="0 0 ${-PI/2}"/>
+      <origin xyz="0 0.115 0" rpy="0 0 ${-pi/2}"/>
       <geometry>
         <mesh filename="package://innok_heros_description/meshes/wheel_tractor_large.STL" />
@@ -48,5 +48,5 @@
     <parent link="drive_box_${front_rear}"/>
     <child link="wheel_${front_rear}_${left_right}"/>
-    <origin xyz="0.063 ${flip_y*flip_z * 0.162} -0.184" rpy="0 0 ${PI/2 - PI/2*flip_y*flip_z }"/>
+    <origin xyz="0.063 ${flip_y*flip_z * 0.162} -0.184" rpy="0 0 ${pi/2 - pi/2*flip_y*flip_z }"/>
     <axis xyz="0 ${flip_y * 1} 0" />
   </joint>
