Commit message: split-up of base_link and beam_link, argument for wheel_separation, swing axle

File: urdf/ROS/heros_diff_drive.xacro (robot description, xacro)
@@ -8,5 +8,5 @@
       <leftJoint>joint_base_wheel_rear_right</leftJoint>
       <rightJoint>joint_base_wheel_rear_left</rightJoint>
-      <wheelSeparation>0.580</wheelSeparation>
+      <wheelSeparation>${wheel_seperation}</wheelSeparation>
       <wheelDiameter>${2*wheel_radius}</wheelDiameter>
       <wheelTorque>130</wheelTorque>

File: urdf/innok_heros_3w.xacro (robot description, xacro)
@@ -15,4 +15,5 @@
   <xacro:property name="wheel_width"  value="0.160" />
   <xacro:property name="wheel_mass"   value="5.4" />
+  <xacro:property name="wheel_seperation" value="0.580" />
   <xacro:property name="camera_link"   value="0.05" />
   <xacro:include filename="$(find innok_heros_description)/urdf/modules/heros_base_link.xacro"/>

File: urdf/innok_heros_3wtractor.xacro (robot description, xacro)
@@ -15,4 +15,5 @@
   <xacro:property name="wheel_width"  value="0.100" />
   <xacro:property name="wheel_mass"   value="5.4" />
+  <xacro:property name="wheel_seperation" value="0.580" />
   <xacro:property name="camera_link"   value="0.05" />
   <xacro:include filename="$(find innok_heros_description)/urdf/modules/heros_base_link.xacro"/>

File: urdf/modules/heros_base_link.xacro (robot description, xacro)
@@ -13,5 +13,6 @@
 <robot xmlns:xacro="http://ros.org/wiki/xacro" name="heros_base_link">
 <xacro:macro name="heros_base_link">
-  <link name="base_link">
+  <link name="base_link"/>
+  <link name="beam_link">
     <inertial>
       <origin xyz="0.40 0 0.02" rpy="0 0 0" /> <mass value="2" />
@@ -20,5 +21,5 @@
     <visual>
       <origin xyz="0 0 0" rpy="0 0 0" />
-      <geometry> <mesh filename="package://innok_heros_description/meshes/base_link.STL" /> </geometry>
+      <geometry> <mesh filename="package://innok_heros_description/meshes/beam.STL" /> </geometry>
       <material name="white">
         <color rgba="1 1 1 1"/>
@@ -30,4 +31,11 @@
     </collision>
   </link>
+  <joint name="beam_joint" type="fixed">
+    <origin
+      xyz="0 0 0" rpy="0 0 0" />
+    <parent link="base_link" />
+    <child link="beam_link" />
+    <axis xyz="0 0 0" />
+  </joint>
 </xacro:macro>
 </robot>

File: urdf/modules/heros_battery.xacro (robot description, xacro)
@@ -38,5 +38,5 @@
     <origin
       xyz="${dx} 0 -0.007" rpy="0 0 0" />
-    <parent link="base_link" />
+    <parent link="beam_link" />
     <child link="${name}" />
     <axis xyz="0 0 0" />

File: urdf/modules/heros_caster.xacro (robot description, xacro)
@@ -37,5 +37,5 @@
   <joint name="caster_top_joint" type="fixed">
     <origin xyz="${dx} 0 -0.006" rpy="0 0 0" />
-    <parent link="base_link" />
+    <parent link="beam_link" />
     <child link="caster_top" />
     <axis xyz="0 0 0" />

File: urdf/modules/heros_drive.xacro (robot description, xacro)
@@ -39,5 +39,5 @@
   <joint name="drive_box_joint_${front_rear}" type="fixed">
     <origin xyz="${dx} 0 -0.0065" rpy="0 0 ${PI/2 - PI/2*flip_z }" />
-    <parent link="base_link" />
+    <parent link="beam_link" />
     <child link="drive_box_${front_rear}" />
     <axis xyz="0 0 0" />

File: urdf/modules/heros_mounting_plate.xacro (robot description, xacro)
@@ -38,5 +38,5 @@
   <joint name="mounting_plate_joint" type="fixed">
     <origin xyz=" ${dx} 0 0.05" rpy="0 0 0" />
-    <parent link="base_link" />
+    <parent link="beam_link" />
     <child link="mounting_plate" />
     <axis xyz="0 0 0" />

File: urdf/modules/heros_wheel.xacro (robot description, xacro)
@@ -37,6 +37,6 @@
   <gazebo reference="wheel_${front_rear}_${left_right}">
     <gravity>true</gravity>
-    <mu1>5</mu1>
-    <mu2>5</mu2>
+    <mu1>10</mu1>
+    <mu2>10</mu2>
     <kd>1</kd>
     <kp>10000000000.0</kp>

File: urdf/modules/heros_wheel_tractor_large.xacro (robot description, xacro)
@@ -21,7 +21,7 @@
     </collision>
     <visual>
-      <origin xyz="0 0.115 0" rpy="${-PI/2} 0 0"/>
+      <origin xyz="0 0.115 0" rpy="0 0 ${-PI/2}"/>
       <geometry>
-        <mesh filename="package://innok_heros_description/meshes/wheel_tractor.STL" />
+        <mesh filename="package://innok_heros_description/meshes/wheel_tractor_large.STL" />
       </geometry>
       <material name="">
