Commit message: using libgazebo ros control interface

File: urdf/ROS/heros_diff_drive.xacro (robot description, xacro)
@@ -2,10 +2,12 @@
 <robot xmlns:xacro="http://ros.org/wiki/xacro" name="heros_diff_drive">
 <xacro:macro name="heros_diff_drive" >
-  <gazebo>
-    <plugin name="differential_drive_controller" filename="libgazebo_ros_diff_drive.so">
-      <alwaysOn>true</alwaysOn>
-      <updateRate>100</updateRate>
-      <leftJoint>joint_base_wheel_rear_left</leftJoint>
-      <rightJoint>joint_base_wheel_rear_right</rightJoint>
+<gazebo>
+  <plugin name="differential_drive_controller" filename="libgazebo_ros_diff_drive.so">
+    <alwaysOn>true</alwaysOn>
+    <legacyMode>false</legacyMode>
+    <updateRate>100</updateRate>
+    <robotNamespace>/</robotNamespace>
+      <leftJoint>joint_base_wheel_rear_right</leftJoint>
+      <rightJoint>joint_base_wheel_rear_left</rightJoint>
       <wheelSeparation>${wheel_seperation}</wheelSeparation>
       <wheelDiameter>${2*wheel_radius}</wheelDiameter>
@@ -14,7 +16,16 @@
       <odometryTopic>odom</odometryTopic>
       <robotBaseFrame>base_link</robotBaseFrame>
-      <legacyMode>false</legacyMode>
-    </plugin>
-  </gazebo>
+    <torque>36.9</torque>
+    <odometryFrame>odom</odometryFrame>
+    <odometrySource>world</odometrySource>
+    <publishTf>1</publishTf>
+    <rosDebugLevel>na</rosDebugLevel>
+    <wheelAcceleration>0</wheelAcceleration>
+    <wheelTorque>5</wheelTorque>
+    <robotBaseFrame>base_link</robotBaseFrame>
+    <publishWheelTF>false</publishWheelTF>
+    <publishWheelJointState>false</publishWheelJointState>
+  </plugin>
+</gazebo>
 </xacro:macro>
 </robot>

File: urdf/ROS/heros_joint_pub.xacro (robot description, xacro)
@@ -1,4 +1,4 @@
 <?xml version="1.0"?>
-<robot xmlns:xacro="http://ros.org/wiki/xacro" name="heros_joint_pub">
+<robot xmlns:xacro="http://www.ros.org/wiki/xacro" name="heros_joint_pub">
 <xacro:macro name="heros_joint_pub" params="joints">
   <gazebo>

File: urdf/innok_heros.xacro (robot description, xacro)
@@ -1,12 +1,11 @@
 <?xml version="1.0"?>
 <robot name="innok_heros_full" xmlns:xacro="http://www.ros.org/wiki/xacro">
-  <xacro:arg name="wheel_number" default="3" />
-  <xacro:arg name="wheel_kind" default="0" />
-  <xacro:arg name="swing_axle" default="true" />
+  <xacro:arg name="wheel_kind" default="default" /> <!-- default | tractor | tractor_large -->
+  <xacro:arg name="front_kind" default="swing_axle" /> <!-- swing_axle | caster | 4wd -->
   <!-- constants-->
   <xacro:include filename="$(find innok_heros_description)/urdf/constants.xacro"/>
   <!-- heros base-->
   <xacro:include filename="$(find innok_heros_description)/urdf/innok_heros_universal.xacro"/>
-  <xacro:innok_heros_universal wheel_number='$(arg wheel_number)' swing_axle='$(arg swing_axle)' wheel_kind='$(arg wheel_kind)'/>
-  <update_rate>1</update_rate>
+  <xacro:innok_heros front_kind='$(arg front_kind)' wheel_kind='$(arg wheel_kind)'/>
+   <update_rate>1</update_rate>
 </robot>

File: urdf/innok_heros_universal.xacro (robot description, xacro)
@@ -11,70 +11,29 @@
 -->
 <robot name="innok_heros_universal" xmlns:xacro="http://www.ros.org/wiki/xacro">
-<xacro:macro name="innok_heros_universal" params="wheel_number wheel_kind swing_axle">
+  <xacro:macro name="innok_heros" params="front_kind wheel_kind">
   <material name="Grey">
     <color rgba="0.66 0.66 0.66 1"/>
   </material>
-<!-- Defining xacro properties -->
+  <!-- Defining xacro properties -->
   <xacro:property name="PI" value="3.1415926535897931"/>
   <xacro:property name="wheel_seperation" value="0.580" />
-  <xacro:property name="wheel_number_prop"   value="${wheel_number}"/>
-  <xacro:property name="wheel_kind_prop"   value="${wheel_kind}"/>
-  <!-- Wheel specifications -->
-  <xacro:if value="${wheel_kind_prop == 0}">
-    <xacro:property name="wheel_radius" value="0.160" />
-    <xacro:property name="wheel_width"  value="0.160" />
-    <xacro:property name="wheel_mass"   value="5.4" />
-    <xacro:include filename="$(find innok_heros_description)/urdf/modules/heros_wheel.xacro"/>
-  </xacro:if>
-  <xacro:if value="${wheel_kind_prop == 1}">
-    <xacro:property name="wheel_radius" value="0.200" />
-    <xacro:property name="wheel_width"  value="0.100" />
-    <xacro:property name="wheel_mass"   value="5.4" />
-    <xacro:include filename="$(find innok_heros_description)/urdf/modules/heros_wheel_tractor.xacro" />
-  </xacro:if>
-  <xacro:if value="${wheel_kind_prop == 2}">
-    <xacro:property name="wheel_radius" value="0.300" />
-    <xacro:property name="wheel_width"  value="0.200" />
-    <xacro:property name="wheel_mass"   value="5.4" />
-    <xacro:include filename="$(find innok_heros_description)/urdf/modules/heros_wheel_tractor_large.xacro" />
-  </xacro:if>
-<!-- Including non optional .xacro files -->
+  <xacro:property name="camera_link" value="0.05" />
+  <!-- Including non optional .xacro files -->
   <xacro:include filename="$(find innok_heros_description)/urdf/modules/heros_base_link.xacro"/>
   <xacro:include filename="$(find innok_heros_description)/urdf/modules/heros_drive.xacro" />
   <xacro:include filename="$(find innok_heros_description)/urdf/modules/heros_battery.xacro" />
   <xacro:include filename="$(find innok_heros_description)/urdf/modules/heros_mounting_plate.xacro" />
-<!-- Including wheel number specific .xacro files (choosen in .launch file)... -->
-<!-- ... and declaring wheel number specific macros with its parameters -->
-  <xacro:if value="${wheel_number_prop == 3}">
-    <xacro:include filename="$(find innok_heros_description)/urdf/ROS/heros_joint_pub.xacro" />
-    <xacro:include filename="$(find innok_heros_description)/urdf/ROS/heros_diff_drive.xacro" />
-    <xacro:heros_base_link   							/>
-    <xacro:heros_drive   	  front_rear='rear'     dx='0.018' flip_z='1' wheel_kind='${wheel_kind_prop}'/>
-    <xacro:heros_battery 	  name='battery_box'    dx='0.336'		/>
-    <xacro:heros_mounting_plate   wheels='${wheel_number_prop}'   dx='-0.02'		/>
-    <xacro:heros_diff_drive 							/>
-    <!-- Front wheel configuration: Swing axle or caster -->
-    <xacro:if value="${swing_axle}">
-        <xacro:include filename="$(find innok_heros_description)/urdf/modules/heros_swing_axle.xacro" />
-        <xacro:heros_swing_axle 	 	         	dx='1.02'		/>
-        <xacro:heros_joint_pub joints='joint_base_wheel_rear_left, joint_base_wheel_rear_right, caster_wheel_left_joint, caster_wheel_right_joint, swing_axle_joint, caster_left_joint, caster_right_joint'/>
-    </xacro:if>
-    <xacro:unless value="${swing_axle}">
-        <xacro:include filename="$(find innok_heros_description)/urdf/modules/heros_caster.xacro" />
-        <xacro:heros_caster  	 	         	dx='0.637'		/>
-        <xacro:heros_joint_pub joints='joint_base_wheel_rear_left, joint_base_wheel_rear_right, caster_bot_joint, caster_wheel_joint'					/>
-    </xacro:unless>
-  </xacro:if>
-  <xacro:if value="${wheel_number_prop == 4}">
-    <xacro:include filename="$(find innok_heros_description)/urdf/ROS/heros_joint_pub.xacro" />
-    <xacro:include filename="$(find innok_heros_description)/urdf/ROS/heros_skid_drive.xacro" />
-    <xacro:heros_base_link   							/>
-    <xacro:heros_drive   	  front_rear='front'     dx='0.782' flip_z='-1' wheel_kind='${wheel_kind_prop}'/>
-    <xacro:heros_drive   	  front_rear='rear'     dx='0.018' flip_z='1' wheel_kind='${wheel_kind_prop}'/>
-    <xacro:heros_battery 	  name='battery_box'    dx='0.336'		/>
-    <xacro:heros_mounting_plate   wheels='${wheel_number_prop}'		dx='-0.02'		/>
-    <xacro:heros_joint_pub joints='joint_base_wheel_rear_left, joint_base_wheel_rear_right, joint_base_wheel_front_left, joint_base_wheel_front_right'		/>
-    <xacro:heros_skid_drive 							/>
-  </xacro:if>
-</xacro:macro>
+  <!-- Including modules -->
+  <xacro:include filename="$(find innok_heros_description)/urdf/ROS/heros_joint_pub.xacro" />
+  <!-- Wheel specifications -->
+  <xacro:include filename="$(find innok_heros_description)/urdf/configurations/wheel_${wheel_kind}_properties.xacro" />
+  <!-- heros front -->
+  <xacro:include filename="$(find innok_heros_description)/urdf/configurations/front_${front_kind}.xacro" />
+  <!-- Including optional .xacro files (choosen in .launch file) -->
+  <!-- instantiating macros -->
+  <xacro:heros_base_link/>
+  <xacro:heros_drive front_rear='rear' dx='0.018' flip_z='1'/>
+  <xacro:heros_battery name='battery_box' dx='0.336'/>
+  <xacro:heros_front/>
+  </xacro:macro>
 </robot>

File: urdf/modules/heros_base_link.xacro (robot description, xacro)
@@ -3,7 +3,7 @@
 Description of the base module for the Innok Heros mobile platform.
 Software License Agreement (BSD)
-\authors Jonathan Hechtbauer
+\authors Tobias Griepentrog
 \maintainer Sabrina Heerklotz <sh@innok-robotics.de>
-\copyright Copyright (c) 2015, Innok Robotics GmbH, All rights reserved
+\copyright Copyright (c) 2021, Innok Robotics GmbH, All rights reserved
 Redistribution and use in source and binary forms, with or without modification, are permitted provided that the following conditions are met:
 1. Redistributions of source code must retain the above copyright notice, this list of conditions and the following disclaimer.
@@ -11,5 +11,5 @@
 THIS SOFTWARE IS PROVIDED BY THE COPYRIGHT HOLDERS AND CONTRIBUTORS "AS IS" AND ANY EXPRESS OR IMPLIED WARRANTIES, INCLUDING, BUT NOT LIMITED TO, THE IMPLIED WARRANTIES OF MERCHANTABILITY AND FITNESS FOR A PARTICULAR PURPOSE ARE DISCLAIMED. IN NO EVENT SHALL THE COPYRIGHT HOLDER OR CONTRIBUTORS BE LIABLE FOR ANY DIRECT, INDIRECT, INCIDENTAL, SPECIAL, EXEMPLARY, OR CONSEQUENTIAL DAMAGES (INCLUDING, BUT NOT LIMITED TO, PROCUREMENT OF SUBSTITUTE GOODS OR SERVICES; LOSS OF USE, DATA, OR PROFITS; OR BUSINESS INTERRUPTION) HOWEVER CAUSED AND ON ANY THEORY OF LIABILITY, WHETHER IN CONTRACT, STRICT LIABILITY, OR TORT (INCLUDING NEGLIGENCE OR OTHERWISE) ARISING IN ANY WAY OUT OF THE USE OF THIS SOFTWARE, EVEN IF ADVISED OF THE POSSIBILITY OF SUCH DAMAGE.
 -->
-<robot xmlns:xacro="http://ros.org/wiki/xacro" name="heros_base_link">
+<robot xmlns:xacro="http://www.ros.org/wiki/xacro" name="heros_base_link">
 <xacro:macro name="heros_base_link">
   <link name="base_link"/>
@@ -21,5 +21,5 @@
     <visual>
       <origin xyz="0 0 0" rpy="0 0 0" />
-      <geometry> <mesh filename="package://innok_heros_description/meshes/beam.STL" /> </geometry>
+      <geometry> <mesh filename="$(find innok_heros_description)/meshes/beam.STL" /> </geometry>
       <material name="white">
         <color rgba="1 1 1 1"/>

File: urdf/modules/heros_battery.xacro (robot description, xacro)
@@ -3,7 +3,7 @@
 Description of the battery module for the Innok Heros mobile platform.
 Software License Agreement (BSD)
-\authors Jonathan Hechtbauer
+\authors Tobias Griepentrog
 \maintainer Sabrina Heerklotz <sh@innok-robotics.de>
-\copyright Copyright (c) 2015, Innok Robotics GmbH, All rights reserved
+\copyright Copyright (c) 2021, Innok Robotics GmbH, All rights reserved
 Redistribution and use in source and binary forms, with or without modification, are permitted provided that the following conditions are met:
 1. Redistributions of source code must retain the above copyright notice, this list of conditions and the following disclaimer.
@@ -11,5 +11,5 @@
 THIS SOFTWARE IS PROVIDED BY THE COPYRIGHT HOLDERS AND CONTRIBUTORS "AS IS" AND ANY EXPRESS OR IMPLIED WARRANTIES, INCLUDING, BUT NOT LIMITED TO, THE IMPLIED WARRANTIES OF MERCHANTABILITY AND FITNESS FOR A PARTICULAR PURPOSE ARE DISCLAIMED. IN NO EVENT SHALL THE COPYRIGHT HOLDER OR CONTRIBUTORS BE LIABLE FOR ANY DIRECT, INDIRECT, INCIDENTAL, SPECIAL, EXEMPLARY, OR CONSEQUENTIAL DAMAGES (INCLUDING, BUT NOT LIMITED TO, PROCUREMENT OF SUBSTITUTE GOODS OR SERVICES; LOSS OF USE, DATA, OR PROFITS; OR BUSINESS INTERRUPTION) HOWEVER CAUSED AND ON ANY THEORY OF LIABILITY, WHETHER IN CONTRACT, STRICT LIABILITY, OR TORT (INCLUDING NEGLIGENCE OR OTHERWISE) ARISING IN ANY WAY OUT OF THE USE OF THIS SOFTWARE, EVEN IF ADVISED OF THE POSSIBILITY OF SUCH DAMAGE.
 -->
-<robot xmlns:xacro="http://ros.org/wiki/xacro" name="heros_battery">
+<robot xmlns:xacro="http://www.ros.org/wiki/xacro" name="heros_battery">
 <xacro:macro name="heros_battery" params="name dx">>
   <link name="${name}">
@@ -22,5 +22,5 @@
       <origin xyz="0 0 0" rpy="0 0 0" />
       <geometry>
-        <mesh filename="package://innok_heros_description/meshes/battery_box.STL" />
+        <mesh filename="$(find innok_heros_description)/meshes/battery_box.STL" />
       </geometry>
       <material name="white">

File: urdf/modules/heros_caster.xacro (robot description, xacro)
@@ -3,7 +3,7 @@
 Description of the caster module for the Innok Heros mobile platform.
 Software License Agreement (BSD)
-\authors Jonathan Hechtbauer
+\authors Tobias Griepentrog
 \maintainer Sabrina Heerklotz <sh@innok-robotics.de>
-\copyright Copyright (c) 2015, Innok Robotics GmbH, All rights reserved
+\copyright Copyright (c) 2021, Innok Robotics GmbH, All rights reserved
 Redistribution and use in source and binary forms, with or without modification, are permitted provided that the following conditions are met:
 1. Redistributions of source code must retain the above copyright notice, this list of conditions and the following disclaimer.
@@ -11,5 +11,5 @@
 THIS SOFTWARE IS PROVIDED BY THE COPYRIGHT HOLDERS AND CONTRIBUTORS "AS IS" AND ANY EXPRESS OR IMPLIED WARRANTIES, INCLUDING, BUT NOT LIMITED TO, THE IMPLIED WARRANTIES OF MERCHANTABILITY AND FITNESS FOR A PARTICULAR PURPOSE ARE DISCLAIMED. IN NO EVENT SHALL THE COPYRIGHT HOLDER OR CONTRIBUTORS BE LIABLE FOR ANY DIRECT, INDIRECT, INCIDENTAL, SPECIAL, EXEMPLARY, OR CONSEQUENTIAL DAMAGES (INCLUDING, BUT NOT LIMITED TO, PROCUREMENT OF SUBSTITUTE GOODS OR SERVICES; LOSS OF USE, DATA, OR PROFITS; OR BUSINESS INTERRUPTION) HOWEVER CAUSED AND ON ANY THEORY OF LIABILITY, WHETHER IN CONTRACT, STRICT LIABILITY, OR TORT (INCLUDING NEGLIGENCE OR OTHERWISE) ARISING IN ANY WAY OUT OF THE USE OF THIS SOFTWARE, EVEN IF ADVISED OF THE POSSIBILITY OF SUCH DAMAGE.
 -->
-<robot xmlns:xacro="http://ros.org/wiki/xacro" name="heros_caster">
+<robot xmlns:xacro="http://www.ros.org/wiki/xacro" name="heros_caster">
 <xacro:macro name="heros_caster" params="dx">
   <link name="caster_top">
@@ -22,5 +22,5 @@
       <origin xyz="0 0 0" rpy="0 0 0" />
       <geometry>
-        <mesh filename="package://innok_heros_description/meshes/caster_top.STL" />
+        <mesh filename="$(find innok_heros_description)/meshes/caster_top.STL" />
       </geometry>
       <material name="white">
@@ -50,5 +50,5 @@
       <origin xyz="0 0 0" rpy="0 0 0" />
       <geometry>
-        <mesh filename="package://innok_heros_description/meshes/caster_bot.STL" />
+        <mesh filename="$(find innok_heros_description)/meshes/caster_bot.STL" />
       </geometry>
       <material name="white">
@@ -78,5 +78,5 @@
       <origin xyz="0 0 0" rpy="0 0 0" />
       <geometry>
-        <mesh filename="package://innok_heros_description/meshes/caster_wheel.STL" />
+        <mesh filename="$(find innok_heros_description)/meshes/caster_wheel.STL" />
       </geometry>
       <material name="">

File: urdf/modules/heros_drive.xacro (robot description, xacro)
@@ -3,7 +3,7 @@
 Description of the drive module for the Innok Heros mobile platform.
 Software License Agreement (BSD)
-\authors Jonathan Hechtbauer
+\authors Tobias Griepentrog
 \maintainer Sabrina Heerklotz <sh@innok-robotics.de>
-\copyright Copyright (c) 2015, Innok Robotics GmbH, All rights reserved
+\copyright Copyright (c) 2021, Innok Robotics GmbH, All rights reserved
 Redistribution and use in source and binary forms, with or without modification, are permitted provided that the following conditions are met:
 1. Redistributions of source code must retain the above copyright notice, this list of conditions and the following disclaimer.
@@ -11,23 +11,13 @@
 THIS SOFTWARE IS PROVIDED BY THE COPYRIGHT HOLDERS AND CONTRIBUTORS "AS IS" AND ANY EXPRESS OR IMPLIED WARRANTIES, INCLUDING, BUT NOT LIMITED TO, THE IMPLIED WARRANTIES OF MERCHANTABILITY AND FITNESS FOR A PARTICULAR PURPOSE ARE DISCLAIMED. IN NO EVENT SHALL THE COPYRIGHT HOLDER OR CONTRIBUTORS BE LIABLE FOR ANY DIRECT, INDIRECT, INCIDENTAL, SPECIAL, EXEMPLARY, OR CONSEQUENTIAL DAMAGES (INCLUDING, BUT NOT LIMITED TO, PROCUREMENT OF SUBSTITUTE GOODS OR SERVICES; LOSS OF USE, DATA, OR PROFITS; OR BUSINESS INTERRUPTION) HOWEVER CAUSED AND ON ANY THEORY OF LIABILITY, WHETHER IN CONTRACT, STRICT LIABILITY, OR TORT (INCLUDING NEGLIGENCE OR OTHERWISE) ARISING IN ANY WAY OUT OF THE USE OF THIS SOFTWARE, EVEN IF ADVISED OF THE POSSIBILITY OF SUCH DAMAGE.
 -->
-<robot xmlns:xacro="http://ros.org/wiki/xacro" name="heros_drive">
-<xacro:macro name="heros_drive" params="front_rear dx flip_z wheel_kind:=0">
-  <xacro:if value="${wheel_kind == 0}">
-    <xacro:heros_wheel front_rear="${front_rear}" left_right="left"  flip_y="1"  flip_z="${flip_z}"/>
-    <xacro:heros_wheel front_rear="${front_rear}" left_right="right" flip_y="-1" flip_z="${flip_z}"/>
-  </xacro:if>
-  <xacro:if value="${wheel_kind == 1}">
-    <xacro:heros_wheel_tractor front_rear="${front_rear}" left_right="left"  flip_y="1"  flip_z="${flip_z}"/>
-    <xacro:heros_wheel_tractor front_rear="${front_rear}" left_right="right" flip_y="-1" flip_z="${flip_z}"/>
-  </xacro:if>
-  <xacro:if value="${wheel_kind == 2}">
-    <xacro:heros_wheel_tractor_large front_rear="${front_rear}" left_right="left"  flip_y="1"  flip_z="${flip_z}"/>
-    <xacro:heros_wheel_tractor_large front_rear="${front_rear}" left_right="right" flip_y="-1" flip_z="${flip_z}"/>
-  </xacro:if>
+<robot xmlns:xacro="http://www.ros.org/wiki/xacro" name="heros_drive">
+<xacro:macro name="heros_drive" params="front_rear dx flip_z">
+  <xacro:include filename="$(find innok_heros_description)/urdf/modules/heros_wheel.xacro" />
+  <xacro:heros_wheel front_rear="${front_rear}" left_right="left"  flip_y="1"  flip_z="${flip_z}"/>
+  <xacro:heros_wheel front_rear="${front_rear}" left_right="right" flip_y="-1" flip_z="${flip_z}"/>
   <link name="drive_box_${front_rear}">
     <inertial>
       <origin xyz="0.122 -0.0026 -0.136" rpy="0 0 0" />
-       <!--mass value="10.6" /-->
-       <mass value="0.5" />
+       <mass value="10.6" />
       <inertia ixx="0.316" ixy="0" ixz="0" iyy="0.166" iyz="0" izz="0.307" />
     </inertial>
@@ -35,5 +25,5 @@
       <origin xyz="0 0 0" rpy="0 0 0" />
       <geometry>
-        <mesh filename="package://innok_heros_description/meshes/drive_box.STL" />
+        <mesh filename="$(find innok_heros_description)/meshes/drive_box.STL" />
       </geometry>
       <material name="white">

File: urdf/modules/heros_mounting_plate.xacro (robot description, xacro)
@@ -3,7 +3,7 @@
 Description of the mounting plate module for the Innok Heros mobile platform.
 Software License Agreement (BSD)
-\authors Jonathan Hechtbauer
+\authors Tobias Griepentrog
 \maintainer Sabrina Heerklotz <sh@innok-robotics.de>
-\copyright Copyright (c) 2015, Innok Robotics GmbH, All rights reserved
+\copyright Copyright (c) 2021, Innok Robotics GmbH, All rights reserved
 Redistribution and use in source and binary forms, with or without modification, are permitted provided that the following conditions are met:
 1. Redistributions of source code must retain the above copyright notice, this list of conditions and the following disclaimer.
@@ -11,5 +11,5 @@
 THIS SOFTWARE IS PROVIDED BY THE COPYRIGHT HOLDERS AND CONTRIBUTORS "AS IS" AND ANY EXPRESS OR IMPLIED WARRANTIES, INCLUDING, BUT NOT LIMITED TO, THE IMPLIED WARRANTIES OF MERCHANTABILITY AND FITNESS FOR A PARTICULAR PURPOSE ARE DISCLAIMED. IN NO EVENT SHALL THE COPYRIGHT HOLDER OR CONTRIBUTORS BE LIABLE FOR ANY DIRECT, INDIRECT, INCIDENTAL, SPECIAL, EXEMPLARY, OR CONSEQUENTIAL DAMAGES (INCLUDING, BUT NOT LIMITED TO, PROCUREMENT OF SUBSTITUTE GOODS OR SERVICES; LOSS OF USE, DATA, OR PROFITS; OR BUSINESS INTERRUPTION) HOWEVER CAUSED AND ON ANY THEORY OF LIABILITY, WHETHER IN CONTRACT, STRICT LIABILITY, OR TORT (INCLUDING NEGLIGENCE OR OTHERWISE) ARISING IN ANY WAY OUT OF THE USE OF THIS SOFTWARE, EVEN IF ADVISED OF THE POSSIBILITY OF SUCH DAMAGE.
 -->
-<robot xmlns:xacro="http://ros.org/wiki/xacro" name="heros_plate">
+<robot xmlns:xacro="http://www.ros.org/wiki/xacro" name="heros_plate">
 <xacro:macro name="heros_mounting_plate" params="wheels dx">
   <link name="mounting_plate">
@@ -23,5 +23,5 @@
       <origin xyz="0 0 0" rpy="0 0 0" />
       <geometry>
-        <mesh filename="package://innok_heros_description/meshes/mounting_plate_${wheels}w.STL" />
+        <mesh filename="$(find innok_heros_description)/meshes/mounting_plate_${wheels}w.STL" />
       </geometry>
       <material name="white">
