Commit message: using libgazebo ros control interface

File: urdf/modules/heros_swing_axle.xacro (robot description, xacro)
@@ -3,7 +3,7 @@
 Description of the swing axle module for the Innok Heros mobile platform.
 Software License Agreement (BSD)
-\authors Jonathan Hechtbauer
+\authors Tobias Griepentrog
 \maintainer Sabrina Heerklotz <sh@innok-robotics.de>
-\copyright Copyright (c) 2015, Innok Robotics GmbH, All rights reserved
+\copyright Copyright (c) 2021, Innok Robotics GmbH, All rights reserved
 Redistribution and use in source and binary forms, with or without modification, are permitted provided that the following conditions are met:
 1. Redistributions of source code must retain the above copyright notice, this list of conditions and the following disclaimer.
@@ -11,5 +11,5 @@
 THIS SOFTWARE IS PROVIDED BY THE COPYRIGHT HOLDERS AND CONTRIBUTORS "AS IS" AND ANY EXPRESS OR IMPLIED WARRANTIES, INCLUDING, BUT NOT LIMITED TO, THE IMPLIED WARRANTIES OF MERCHANTABILITY AND FITNESS FOR A PARTICULAR PURPOSE ARE DISCLAIMED. IN NO EVENT SHALL THE COPYRIGHT HOLDER OR CONTRIBUTORS BE LIABLE FOR ANY DIRECT, INDIRECT, INCIDENTAL, SPECIAL, EXEMPLARY, OR CONSEQUENTIAL DAMAGES (INCLUDING, BUT NOT LIMITED TO, PROCUREMENT OF SUBSTITUTE GOODS OR SERVICES; LOSS OF USE, DATA, OR PROFITS; OR BUSINESS INTERRUPTION) HOWEVER CAUSED AND ON ANY THEORY OF LIABILITY, WHETHER IN CONTRACT, STRICT LIABILITY, OR TORT (INCLUDING NEGLIGENCE OR OTHERWISE) ARISING IN ANY WAY OUT OF THE USE OF THIS SOFTWARE, EVEN IF ADVISED OF THE POSSIBILITY OF SUCH DAMAGE.
 -->
-<robot xmlns:xacro="http://ros.org/wiki/xacro" name="heros_swing_axle">
+<robot xmlns:xacro="http://www.ros.org/wiki/xacro" name="heros_swing_axle">
 <xacro:macro name="heros_swing_axle" params="dx">
   <link name="swing_axle_top">
@@ -20,5 +20,5 @@
     <visual>
       <origin xyz="0 0 0" rpy="0 0 0" />
-      <geometry> <mesh filename="package://innok_heros_description/meshes/swing_axle_top.STL" /> </geometry>
+      <geometry> <mesh filename="$(find innok_heros_description)/meshes/swing_axle_top.STL" /> </geometry>
       <material name="white">
         <color rgba="1 1 1 1"/>
@@ -48,5 +48,5 @@
       <origin xyz="0 0 0" rpy="0 0 0" />
       <geometry>
-        <mesh filename="package://innok_heros_description/meshes/swing_axle_bot.STL" />
+        <mesh filename="$(find innok_heros_description)/meshes/swing_axle_bot.STL" />
       </geometry>
       <material name="white">
@@ -76,5 +76,5 @@
       <origin xyz="0 0 0" rpy="0 0 0" />
       <geometry>
-        <mesh filename="package://innok_heros_description/meshes/caster_bot.STL" />
+        <mesh filename="$(find innok_heros_description)/meshes/caster_bot.STL" />
       </geometry>
       <material name="white">
@@ -98,5 +98,5 @@
       <origin xyz="0 0 0" rpy="0 0 0" />
       <geometry>
-        <mesh filename="package://innok_heros_description/meshes/caster_wheel.STL" />
+        <mesh filename="$(find innok_heros_description)/meshes/caster_wheel.STL" />
       </geometry>
       <material name="">
@@ -131,5 +131,5 @@
       <origin xyz="0 0 0" rpy="0 0 0" />
       <geometry>
-        <mesh filename="package://innok_heros_description/meshes/caster_bot.STL" />
+        <mesh filename="$(find innok_heros_description)/meshes/caster_bot.STL" />
       </geometry>
       <material name="white">
@@ -153,5 +153,5 @@
       <origin xyz="0 0 0" rpy="0 0 0" />
       <geometry>
-        <mesh filename="package://innok_heros_description/meshes/caster_wheel.STL" />
+        <mesh filename="$(find innok_heros_description)/meshes/caster_wheel.STL" />
       </geometry>
       <material name="">

File: urdf/modules/heros_wheel.xacro (robot description, xacro)
@@ -3,7 +3,7 @@
 Description of the wheel module for the Innok Heros mobile platform.
 Software License Agreement (BSD)
-\authors Jonathan Hechtbauer
+\authors Tobias Griepentrog
 \maintainer Sabrina Heerklotz <sh@innok-robotics.de>
-\copyright Copyright (c) 2015, Innok Robotics GmbH, All rights reserved
+\copyright Copyright (c) 2021, Innok Robotics GmbH, All rights reserved
 Redistribution and use in source and binary forms, with or without modification, are permitted provided that the following conditions are met:
 1. Redistributions of source code must retain the above copyright notice, this list of conditions and the following disclaimer.
@@ -11,5 +11,5 @@
 THIS SOFTWARE IS PROVIDED BY THE COPYRIGHT HOLDERS AND CONTRIBUTORS "AS IS" AND ANY EXPRESS OR IMPLIED WARRANTIES, INCLUDING, BUT NOT LIMITED TO, THE IMPLIED WARRANTIES OF MERCHANTABILITY AND FITNESS FOR A PARTICULAR PURPOSE ARE DISCLAIMED. IN NO EVENT SHALL THE COPYRIGHT HOLDER OR CONTRIBUTORS BE LIABLE FOR ANY DIRECT, INDIRECT, INCIDENTAL, SPECIAL, EXEMPLARY, OR CONSEQUENTIAL DAMAGES (INCLUDING, BUT NOT LIMITED TO, PROCUREMENT OF SUBSTITUTE GOODS OR SERVICES; LOSS OF USE, DATA, OR PROFITS; OR BUSINESS INTERRUPTION) HOWEVER CAUSED AND ON ANY THEORY OF LIABILITY, WHETHER IN CONTRACT, STRICT LIABILITY, OR TORT (INCLUDING NEGLIGENCE OR OTHERWISE) ARISING IN ANY WAY OUT OF THE USE OF THIS SOFTWARE, EVEN IF ADVISED OF THE POSSIBILITY OF SUCH DAMAGE.
 -->
-<robot xmlns:xacro="http://ros.org/wiki/xacro" name="heros_wheel">
+<robot xmlns:xacro="http://www.ros.org/wiki/xacro" name="heros_wheel">
 <xacro:macro name="heros_wheel" params="front_rear left_right flip_y flip_z">
   <link name="wheel_${front_rear}_${left_right}">
@@ -23,5 +23,5 @@
       <origin xyz="0 0 0" rpy="0 0 0"/>
       <geometry>
-        <mesh filename="package://innok_heros_description/meshes/wheel.STL" />
+	      <mesh filename="$(find innok_heros_description)/meshes/${wheel_mesh}" />
       </geometry>
       <material name="">
@@ -40,5 +40,5 @@
     <mu2>10</mu2>
     <kd>1</kd>
-    <kp>10000000000.0</kp>
+    <kp>1000000000.0</kp>
     <fdir1>0 0 1</fdir1>
     <selfCollide>false</selfCollide>
@@ -54,5 +54,5 @@
     <type>transmission_interface/SimpleTransmission</type>
     <joint name="joint_base_wheel_${front_rear}_${left_right}">
-      <hardwareInterface>EffortJointInterface</hardwareInterface>
+    <hardwareInterface>hardware_interface/VelocityJointInterface</hardwareInterface>
     </joint>
     <actuator name="motor_wheel_${front_rear}_${left_right}">
