Commit message: revert mesh file path

File: urdf/modules/heros_base_link.xacro (robot description, xacro)
@@ -21,5 +21,5 @@
     <visual>
       <origin xyz="0 0 0" rpy="0 0 0" />
-      <geometry> <mesh filename="$(find innok_heros_description)/meshes/beam.STL" /> </geometry>
+      <geometry> <mesh filename="package://innok_heros_description/meshes/beam.STL" /> </geometry>
       <material name="white">
         <color rgba="1 1 1 1"/>

File: urdf/modules/heros_battery.xacro (robot description, xacro)
@@ -22,5 +22,5 @@
       <origin xyz="0 0 0" rpy="0 0 0" />
       <geometry>
-        <mesh filename="$(find innok_heros_description)/meshes/battery_box.STL" />
+        <mesh filename="package://innok_heros_description/meshes/battery_box.STL" />
       </geometry>
       <material name="white">

File: urdf/modules/heros_caster.xacro (robot description, xacro)
@@ -22,5 +22,5 @@
       <origin xyz="0 0 0" rpy="0 0 0" />
       <geometry>
-        <mesh filename="$(find innok_heros_description)/meshes/caster_top.STL" />
+        <mesh filename="package://innok_heros_description/meshes/caster_top.STL" />
       </geometry>
       <material name="white">
@@ -50,5 +50,5 @@
       <origin xyz="0 0 0" rpy="0 0 0" />
       <geometry>
-        <mesh filename="$(find innok_heros_description)/meshes/caster_bot.STL" />
+        <mesh filename="package://innok_heros_description/meshes/caster_bot.STL" />
       </geometry>
       <material name="white">
@@ -78,5 +78,5 @@
       <origin xyz="0 0 0" rpy="0 0 0" />
       <geometry>
-        <mesh filename="$(find innok_heros_description)/meshes/caster_wheel.STL" />
+        <mesh filename="package://innok_heros_description/meshes/caster_wheel.STL" />
       </geometry>
       <material name="">

File: urdf/modules/heros_drive.xacro (robot description, xacro)
@@ -25,5 +25,5 @@
       <origin xyz="0 0 0" rpy="0 0 0" />
       <geometry>
-        <mesh filename="$(find innok_heros_description)/meshes/drive_box.STL" />
+        <mesh filename="package://innok_heros_description/meshes/drive_box.STL" />
       </geometry>
       <material name="white">

File: urdf/modules/heros_mounting_plate.xacro (robot description, xacro)
@@ -23,5 +23,5 @@
       <origin xyz="0 0 0" rpy="0 0 0" />
       <geometry>
-        <mesh filename="$(find innok_heros_description)/meshes/mounting_plate_${wheels}w.STL" />
+        <mesh filename="package://innok_heros_description/meshes/mounting_plate_${wheels}w.STL" />
       </geometry>
       <material name="white">

File: urdf/modules/heros_swing_axle.xacro (robot description, xacro)
@@ -20,5 +20,5 @@
     <visual>
       <origin xyz="0 0 0" rpy="0 0 0" />
-      <geometry> <mesh filename="$(find innok_heros_description)/meshes/swing_axle_top.STL" /> </geometry>
+      <geometry> <mesh filename="package://innok_heros_description/meshes/swing_axle_top.STL" /> </geometry>
       <material name="white">
         <color rgba="1 1 1 1"/>
@@ -48,5 +48,5 @@
       <origin xyz="0 0 0" rpy="0 0 0" />
       <geometry>
-        <mesh filename="$(find innok_heros_description)/meshes/swing_axle_bot.STL" />
+        <mesh filename="package://innok_heros_description/meshes/swing_axle_bot.STL" />
       </geometry>
       <material name="white">
@@ -76,5 +76,5 @@
       <origin xyz="0 0 0" rpy="0 0 0" />
       <geometry>
-        <mesh filename="$(find innok_heros_description)/meshes/caster_bot.STL" />
+        <mesh filename="package://innok_heros_description/meshes/caster_bot.STL" />
       </geometry>
       <material name="white">
@@ -98,5 +98,5 @@
       <origin xyz="0 0 0" rpy="0 0 0" />
       <geometry>
-        <mesh filename="$(find innok_heros_description)/meshes/caster_wheel.STL" />
+        <mesh filename="package://innok_heros_description/meshes/caster_wheel.STL" />
       </geometry>
       <material name="">
@@ -131,5 +131,5 @@
       <origin xyz="0 0 0" rpy="0 0 0" />
       <geometry>
-        <mesh filename="$(find innok_heros_description)/meshes/caster_bot.STL" />
+        <mesh filename="package://innok_heros_description/meshes/caster_bot.STL" />
       </geometry>
       <material name="white">
@@ -153,5 +153,5 @@
       <origin xyz="0 0 0" rpy="0 0 0" />
       <geometry>
-        <mesh filename="$(find innok_heros_description)/meshes/caster_wheel.STL" />
+        <mesh filename="package://innok_heros_description/meshes/caster_wheel.STL" />
       </geometry>
       <material name="">

File: urdf/modules/heros_wheel.xacro (robot description, xacro)
@@ -23,5 +23,5 @@
       <origin xyz="0 0 0" rpy="0 0 0"/>
       <geometry>
-	      <mesh filename="$(find innok_heros_description)/meshes/${wheel_mesh}" />
+	      <mesh filename="package://innok_heros_description/meshes/${wheel_mesh}" />
       </geometry>
       <material name="">
